File: _autosave-jr60-1-pcb.kicad_sch (KiCad schematic)
At the start: 1 part

Commit message: init
Parts:
- added C?: C_Small, symbol Device:C_Small
- added R?: R_Small, symbol Device:R_Small
- added SW?: SW_Push, symbol Switch:SW_Push
- added Y?: Crystal_GND24, symbol Device:Crystal_GND24
Changed lines of the file:
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@@
 (kicad_sch (version 20211123) (generator eeschema)
   (paper "A4")
+  (symbol (lib_id "Switch:SW_Push") (at 76.2 58.42 0) (unit 1)
+    (in_bom yes) (on_board yes) (fields_autoplaced)
+    (property "Reference" "SW?" (id 0) (at 76.2 50.8 0))
+    (property "Value" "SW_Push" (id 1) (at 76.2 53.34 0))
+    (property "Footprint" "" (id 2) (at 76.2 53.34 0)
+      (effects (font (size 1.27 1.27)) hide)
+    )
+    (property "Datasheet" "~" (id 3) (at 76.2 53.34 0)
+      (effects (font (size 1.27 1.27)) hide)
+    )
+    (pin "1")
+    (pin "2")
+  )
+  (symbol (lib_id "Device:C_Small") (at 87.63 71.12 0) (unit 1)
+    (in_bom yes) (on_board yes) (fields_autoplaced)
+    (property "Reference" "C?" (id 0) (at 90.17 69.8562 0)
+      (effects (font (size 1.27 1.27)) (justify left))
+    )
+    (property "Value" "C_Small" (id 1) (at 90.17 72.3962 0)
+      (effects (font (size 1.27 1.27)) (justify left))
+    )
+    (property "Footprint" "" (id 2) (at 87.63 71.12 0)
+      (effects (font (size 1.27 1.27)) hide)
+    )
+    (property "Datasheet" "~" (id 3) (at 87.63 71.12 0)
+      (effects (font (size 1.27 1.27)) hide)
+    )
+    (pin "1")
+    (pin "2")
+  )
+  (symbol (lib_id "Device:R_Small") (at 97.79 59.69 0) (unit 1)
+    (in_bom yes) (on_board yes) (fields_autoplaced)
+    (property "Reference" "R?" (id 0) (at 100.33 58.4199 0)
+      (effects (font (size 1.27 1.27)) (justify left))
+    )
+    (property "Value" "R_Small" (id 1) (at 100.33 60.9599 0)
+      (effects (font (size 1.27 1.27)) (justify left))
+    )
+    (property "Footprint" "" (id 2) (at 97.79 59.69 0)
+      (effects (font (size 1.27 1.27)) hide)
+    )
+    (property "Datasheet" "~" (id 3) (at 97.79 59.69 0)
+      (effects (font (size 1.27 1.27)) hide)
+    )
+    (pin "1")
+    (pin "2")
+  )
   (symbol (lib_id "MCU_Microchip_ATmega:ATmega32U4-A") (at 148.59 93.98 0) (unit 1)
     (in_bom yes) (on_board yes) (fields_autoplaced)
@@
     (pin "9")
   )
+  (symbol (lib_id "Device:Crystal_GND24") (at 102.87 77.47 0) (unit 1)
+    (in_bom yes) (on_board yes) (fields_autoplaced)
+    (property "Reference" "Y?" (id 0) (at 114.3 73.8886 0))
+    (property "Value" "Crystal_GND24" (id 1) (at 114.3 76.4286 0))
+    (property "Footprint" "" (id 2) (at 102.87 77.47 0)
+      (effects (font (size 1.27 1.27)) hide)
+    )
+    (property "Datasheet" "~" (id 3) (at 102.87 77.47 0)
+      (effects (font (size 1.27 1.27)) hide)
+    )
+    (pin "1")
+    (pin "2")
+    (pin "3")
+    (pin "4")
+  )
   (sheet_instances
     (path "/" (page "1"))
   )
   (symbol_instances
+    (path "/44c08b1f-bc34-4943-b3aa-cbe434816179"
+      (reference "C?") (unit 1) (value "C_Small") (footprint "")
+    )
+    (path "/7474c6e7-f34b-44e9-b6ee-ea6989b5dd25"
+      (reference "R?") (unit 1) (value "R_Small") (footprint "")
+    )
+    (path "/411d320c-55ef-4b70-b8a7-1e0d28ffc3e4"
+      (reference "SW?") (unit 1) (value "SW_Push") (footprint "")
+    )
     (path "/b446cb42-d684-471b-97b2-a6cda51b57db"
       (reference "U?") (unit 1) (value "ATmega32U4-A") (footprint "Package_QFP:TQFP-44_10x10mm_P0.8mm")
     )
+    (path "/e041d5e9-7585-43ef-a3d0-5e80b243ef15"
+      (reference "Y?") (unit 1) (value "Crystal_GND24") (footprint "")
+    )
   )
