File: jr60-1-pcb.kicad_sch (KiCad schematic)
At the start: 1 part

Commit message: savepoint
Parts:
- added C?: C_Small, symbol Device:C_Small
- added D? (x2): SMF9V0A, Diode_SMD:D_SMF, symbol Diode:SMF9V0A
- added F?: Polyfuse_Small, symbol Device:Polyfuse_Small
- added R?: R_Small, symbol Device:R_Small
- added SW?: SW_Push, symbol Switch:SW_Push
- added U?: TPD4E05U06DQAR, symbol random-keyboard-parts:TPD4E05U06DQAR
- added USB?: HRO-TYPE-C-31-M-12, symbol Type-C:HRO-TYPE-C-31-M-12
- added Y?: Crystal_GND24, symbol Device:Crystal_GND24
Connections:
- net at U?.13 (~{RESET}): now also R?.2, SW?.2
- net at U?.16 (XTAL2): now also Y?.3
- net at U?.17 (XTAL1): now also Y?.1
- no-connect marks 0 -> 2
Other:
- added sheet Matrix (Matrix.kicad_sch)
Changed lines of the file:
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@@
 (kicad_sch (version 20211123) (generator eeschema)
   (paper "A4")
+  (junction (at 129.54 55.88) (diameter 0) (color 0 0 0 0)
+  )
+  (no_connect (at 64.77 113.03))
+  (no_connect (at 64.77 97.79))
+  (wire (pts (xy 111.76 59.69) (xy 133.35 59.69))
+    (stroke (width 0) (type default) (color 0 0 0 0))
+  )
+  (wire (pts (xy 129.54 55.88) (xy 133.35 55.88))
+    (stroke (width 0) (type default) (color 0 0 0 0))
+  )
+  (wire (pts (xy 124.46 55.88) (xy 129.54 55.88))
+    (stroke (width 0) (type default) (color 0 0 0 0))
+  )
+  (wire (pts (xy 129.54 48.26) (xy 129.54 55.88))
+    (stroke (width 0) (type default) (color 0 0 0 0))
+  )
+  (wire (pts (xy 133.35 67.31) (xy 133.35 66.04))
+    (stroke (width 0) (type default) (color 0 0 0 0))
+  )
+  (wire (pts (xy 111.76 67.31) (xy 133.35 67.31))
+    (stroke (width 0) (type default) (color 0 0 0 0))
+  )
+  (wire (pts (xy 133.35 59.69) (xy 133.35 60.96))
+    (stroke (width 0) (type default) (color 0 0 0 0))
+  )
+  (symbol (lib_id "Switch:SW_Push") (at 119.38 55.88 0) (unit 1)
+    (in_bom yes) (on_board yes) (fields_autoplaced)
+    (property "Reference" "SW?" (id 0) (at 119.38 48.26 0))
+    (property "Value" "SW_Push" (id 1) (at 119.38 50.8 0))
+    (property "Footprint" "" (id 2) (at 119.38 50.8 0)
+      (effects (font (size 1.27 1.27)) hide)
+    )
+    (property "Datasheet" "~" (id 3) (at 119.38 50.8 0)
+      (effects (font (size 1.27 1.27)) hide)
+    )
+    (pin "1")
+    (pin "2")
+  )
+  (symbol (lib_id "Type-C:HRO-TYPE-C-31-M-12") (at 62.23 106.68 0) (unit 1)
+    (in_bom yes) (on_board yes) (fields_autoplaced)
+    (property "Reference" "USB?" (id 0) (at 56.515 86.36 0)
+      (effects (font (size 1.524 1.524)))
+    )
+    (property "Value" "HRO-TYPE-C-31-M-12" (id 1) (at 56.515 90.17 0)
+      (effects (font (size 1.524 1.524)))
+    )
+    (property "Footprint" "" (id 2) (at 62.23 106.68 0)
+      (effects (font (size 1.524 1.524)) hide)
+    )
+    (property "Datasheet" "" (id 3) (at 62.23 106.68 0)
+      (effects (font (size 1.524 1.524)) hide)
+    )
+    (pin "1")
+    (pin "10")
+    (pin "11")
+    (pin "12")
+    (pin "13")
+    (pin "2")
+    (pin "3")
+    (pin "4")
+    (pin "5")
+    (pin "6")
+    (pin "7")
+    (pin "8")
+    (pin "9")
+  )
+  (symbol (lib_id "Device:C_Small") (at 87.63 71.12 0) (unit 1)
+    (in_bom yes) (on_board yes) (fields_autoplaced)
+    (property "Reference" "C?" (id 0) (at 90.17 69.8562 0)
+      (effects (font (size 1.27 1.27)) (justify left))
+    )
+    (property "Value" "C_Small" (id 1) (at 90.17 72.3962 0)
+      (effects (font (size 1.27 1.27)) (justify left))
+    )
+    (property "Footprint" "" (id 2) (at 87.63 71.12 0)
+      (effects (font (size 1.27 1.27)) hide)
+    )
+    (property "Datasheet" "~" (id 3) (at 87.63 71.12 0)
+      (effects (font (size 1.27 1.27)) hide)
+    )
+    (pin "1")
+    (pin "2")
+  )
+  (symbol (lib_id "Diode:SMF9V0A") (at 50.8 138.43 90) (unit 1)
+    (in_bom yes) (on_board yes) (fields_autoplaced)
+    (property "Reference" "D?" (id 0) (at 44.45 138.43 0))
+    (property "Value" "SMF9V0A" (id 1) (at 46.99 138.43 0))
+    (property "Footprint" "Diode_SMD:D_SMF" (id 2) (at 55.88 138.43 0)
+      (effects (font (size 1.27 1.27)) hide)
+    )
+    (property "Datasheet" "https://www.vishay.com/doc?85881" (id 3) (at 50.8 139.7 0)
+      (effects (font (size 1.27 1.27)) hide)
+    )
+    (pin "1")
+    (pin "2")
+  )
+  (symbol (lib_id "Diode:SMF9V0A") (at 50.8 140.97 270) (unit 1)
+    (in_bom yes) (on_board yes) (fields_autoplaced)
+    (property "Reference" "D?" (id 0) (at 44.45 140.97 0))
+    (property "Value" "SMF9V0A" (id 1) (at 46.99 140.97 0))
+    (property "Footprint" "Diode_SMD:D_SMF" (id 2) (at 45.72 140.97 0)
+      (effects (font (size 1.27 1.27)) hide)
+    )
+    (property "Datasheet" "https://www.vishay.com/doc?85881" (id 3) (at 50.8 139.7 0)
+      (effects (font (size 1.27 1.27)) hide)
+    )
+    (pin "1")
+    (pin "2")
+  )
+  (symbol (lib_id "Device:R_Small") (at 129.54 45.72 0) (unit 1)
+    (in_bom yes) (on_board yes) (fields_autoplaced)
+    (property "Reference" "R?" (id 0) (at 132.08 44.4499 0)
+      (effects (font (size 1.27 1.27)) (justify left))
+    )
+    (property "Value" "R_Small" (id 1) (at 132.08 46.9899 0)
+      (effects (font (size 1.27 1.27)) (justify left))
+    )
+    (property "Footprint" "" (id 2) (at 129.54 45.72 0)
+      (effects (font (size 1.27 1.27)) hide)
+    )
+    (property "Datasheet" "~" (id 3) (at 129.54 45.72 0)
+      (effects (font (size 1.27 1.27)) hide)
+    )
+    (pin "1")
+    (pin "2")
+  )
+  (symbol (lib_id "Device:Polyfuse_Small") (at 64.77 138.43 0) (unit 1)
+    (in_bom yes) (on_board yes) (fields_autoplaced)
+    (property "Reference" "F?" (id 0) (at 67.31 137.1599 0)
+      (effects (font (size 1.27 1.27)) (justify left))
+    )
+    (property "Value" "Polyfuse_Small" (id 1) (at 67.31 139.6999 0)
+      (effects (font (size 1.27 1.27)) (justify left))
+    )
+    (property "Footprint" "" (id 2) (at 66.04 143.51 0)
+      (effects (font (size 1.27 1.27)) (justify left) hide)
+    )
+    (property "Datasheet" "~" (id 3) (at 64.77 138.43 0)
+      (effects (font (size 1.27 1.27)) hide)
+    )
+    (pin "1")
+    (pin "2")
+  )
   (symbol (lib_id "MCU_Microchip_ATmega:ATmega32U4-A") (at 148.59 93.98 0) (unit 1)
     (in_bom yes) (on_board yes) (fields_autoplaced)
@@
     (pin "9")
   )
+  (symbol (lib_id "random-keyboard-parts:TPD4E05U06DQAR") (at 105.41 120.65 180) (unit 1)
+    (in_bom yes) (on_board yes) (fields_autoplaced)
+    (property "Reference" "U?" (id 0) (at 106.045 101.6 0))
+    (property "Value" "TPD4E05U06DQAR" (id 1) (at 106.045 104.14 0))
+    (property "Footprint" "" (id 2) (at 111.76 125.73 0)
+      (effects (font (size 1.27 1.27)) hide)
+    )
+    (property "Datasheet" "" (id 3) (at 111.76 125.73 0)
+      (effects (font (size 1.27 1.27)) hide)
+    )
+    (pin "1")
+    (pin "10")
+    (pin "2")
+    (pin "3")
+    (pin "4")
+    (pin "5")
+    (pin "6")
+    (pin "7")
+    (pin "8")
+    (pin "9")
+  )
+  (symbol (lib_id "Device:Crystal_GND24") (at 111.76 63.5 270) (unit 1)
+    (in_bom yes) (on_board yes) (fields_autoplaced)
+    (property "Reference" "Y?" (id 0) (at 124.46 58.0388 90))
+    (property "Value" "Crystal_GND24" (id 1) (at 124.46 60.5788 90))
+    (property "Footprint" "" (id 2) (at 111.76 63.5 0)
+      (effects (font (size 1.27 1.27)) hide)
+    )
+    (property "Datasheet" "~" (id 3) (at 111.76 63.5 0)
+      (effects (font (size 1.27 1.27)) hide)
+    )
+    (pin "1")
+    (pin "2")
+    (pin "3")
+    (pin "4")
+  )
+  (sheet (at 90.17 162.56) (size 49.53 11.43) (fields_autoplaced)
+    (stroke (width 0.1524) (type solid) (color 0 0 0 0))
+    (fill (color 0 0 0 0.0000))
+    (property "Sheet name" "Matrix" (id 0) (at 90.17 161.8484 0)
+      (effects (font (size 1.27 1.27)) (justify left bottom))
+    )
+    (property "Sheet file" "Matrix.kicad_sch" (id 1) (at 90.17 174.5746 0)
+      (effects (font (size 1.27 1.27)) (justify left top))
+    )
+  )
   (sheet_instances
     (path "/" (page "1"))
+    (path "/2adb9db3-6a14-43dc-bad9-4f0723810605" (page "2"))
   )
   (symbol_instances
+    (path "/44c08b1f-bc34-4943-b3aa-cbe434816179"
+      (reference "C?") (unit 1) (value "C_Small") (footprint "")
+    )
+    (path "/49e3f707-911d-4369-aa33-eef1bfdf9189"
+      (reference "D?") (unit 1) (value "SMF9V0A") (footprint "Diode_SMD:D_SMF")
+    )
+    (path "/6c534d5b-b35e-4c2f-a289-15b19773be5c"
+      (reference "D?") (unit 1) (value "SMF9V0A") (footprint "Diode_SMD:D_SMF")
+    )
+    (path "/2adb9db3-6a14-43dc-bad9-4f0723810605/e189616c-2a1d-43f7-b77e-c08613a720cf"
+      (reference "D?") (unit 1) (value "D_Small") (footprint "")
+    )
+    (path "/86ef4b21-8017-4ae1-b2e1-bb668763f13c"
+      (reference "F?") (unit 1) (value "Polyfuse_Small") (footprint "")
+    )
+    (path "/2adb9db3-6a14-43dc-bad9-4f0723810605/3ff003a8-163b-48c2-859b-a79bfc30ad25"
+      (reference "MX?") (unit 1) (value "MX-NoLED") (footprint "")
+    )
+    (path "/7474c6e7-f34b-44e9-b6ee-ea6989b5dd25"
+      (reference "R?") (unit 1) (value "R_Small") (footprint "")
+    )
+    (path "/411d320c-55ef-4b70-b8a7-1e0d28ffc3e4"
+      (reference "SW?") (unit 1) (value "SW_Push") (footprint "")
+    )
     (path "/b446cb42-d684-471b-97b2-a6cda51b57db"
       (reference "U?") (unit 1) (value "ATmega32U4-A") (footprint "Package_QFP:TQFP-44_10x10mm_P0.8mm")
     )
-  )
+    (path "/c251dd43-6b12-4527-a04a-243deacb1dae"
+      (reference "U?") (unit 1) (value "TPD4E05U06DQAR") (footprint "")
+    )
+    (path "/4198a1aa-4e4f-4856-9cf2-b6ce08ed20de"
+      (reference "USB?") (unit 1) (value "HRO-TYPE-C-31-M-12") (footprint "")
+    )
+    (path "/e041d5e9-7585-43ef-a3d0-5e80b243ef15"
+      (reference "Y?") (unit 1) (value "Crystal_GND24") (footprint "")
+    )
+  )

Commit message: matrix done
Parts:
- removed C?: C_Small, symbol Device:C_Small
- removed D? (x2): SMF9V0A, Diode_SMD:D_SMF, symbol Diode:SMF9V0A
- added C? (x3): 0.1uF, symbol Device:C_Small
- added C?: 1uF, symbol Device:C_Small
- added C? (x2): 22pF, symbol Device:C_Small
- added C?: 10uF, symbol Device:C_Small
- added D?: D_TVS, symbol Device:D_TVS
- added J?: AVR-ISP-6, symbol Connector:AVR-ISP-6
- added R?: 10k, symbol Device:R_Small
- added R? (x2): 22, symbol Device:R_Small
- added R? (x2): 5.1k, symbol Device:R_Small
- R?: value R_Small -> 10k
- Y?: value Crystal_GND24 -> 16MHz
Connections:
- net GND: now reaches SW?.1
- net GND: now also U?.15 (GND), U?.23 (GND), U?.3 (GND), U?.35 (GND), U?.43 (GND), U?.5 (UGND), U?.8 (GND), USB?.1 (GND), USB?.12 (GND), USB?.13 (SHIELD), Y?.2, Y?.4, C?.1, C?.1, C?.2, C?.2, C?.2, C?.2, C?.2, D?.1 (A1), J?.6 (GND), R?.2, R?.2, R?.2
- net RESET: now reaches R?.2, SW?.2, U?.13 (~{RESET})
- net RESET: now also J?.5 (~{RST})
- net at USB?.10 (CC2): now also R?.1
- net at USB?.11 (VBUS): now also F?.1, USB?.2 (VBUS)
- net at USB?.4 (CC1): now also R?.1
- net D-: now reaches USB?.5 (DN2)
- net D-: now also U?.2 (D1-), U?.5 (D2-), U?.6 (NC), U?.9 (NC), USB?.7 (DN1), R?.1
- net D+: now reaches USB?.6 (DP1)
- net D+: now also U?.1 (D1+), U?.10 (NC), U?.4 (D2+), U?.7 (NC), USB?.8 (DP2), R?.1
- net +5V: now reaches R?.1
- net +5V: now also U?.14 (VCC), U?.2 (UVCC), U?.24 (AVCC), U?.34 (VCC), U?.44 (AVCC), U?.7 (VBUS), C?.1, C?.1, C?.1, C?.1, J?.2 (VCC)
- net VCC: now reaches F?.2
- net VCC: now also D?.2 (A2)
- net MOSI: now reaches U?.10 (PB2)
- net MOSI: now also J?.4 (MOSI)
- net MISO: now reaches U?.11 (PB3)
- net MISO: now also J?.1 (MISO)
- net XTAL2: now reaches U?.16 (XTAL2), Y?.3
- net XTAL2: now also C?.2
- net XTAL1: now reaches U?.17 (XTAL1), Y?.1
- net XTAL1: now also C?.2
- net at U?.3 (D-): now also R?.2
- net at U?.33 (~{HWB}/PE2): now also R?.1
- net at U?.4 (D+): now also R?.2
- net at U?.6 (UCAP): now also C?.1
- net SCK: now reaches U?.9 (PB1)
- net SCK: now also J?.3 (SCK)
- no-connect marks 2 -> 3
Other:
- moved on the sheet: F?, R?, SW?, U?, USB?, Y?
